File: BIT3.kicad_pcb (KiCad board)
At the start: 2 copper layers, 121.3 x 109.4 mm, 40 parts, among them J1 Conn_02x04_Odd_Even, J2 Conn_01x02_Pin, Q1 2SC1815, SW1 SW_SPDT, SW2 SW_Push, SW3 SW_Push, U2 SG-107F, U3 SG-107F, U4 SG-107F, U5 SG-107F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

Commit message: Update PCB Design
Parts:
- added R17: R, Resistor_THT:R_Axial_DIN0204_L3.6mm_D1.6mm_P7.62mm_Horizontal, F.Cu at (127.0, 82.5)
- added R18: R, Resistor_THT:R_Axial_DIN0204_L3.6mm_D1.6mm_P7.62mm_Horizontal, F.Cu at (129.5, 74.9)
- added R19: R, Resistor_THT:R_Axial_DIN0204_L3.6mm_D1.6mm_P7.62mm_Horizontal, F.Cu at (132.1, 82.5)
- added R20: R, Resistor_THT:R_Axial_DIN0204_L3.6mm_D1.6mm_P7.62mm_Horizontal, F.Cu at (134.6, 74.9)
- added R21: R, Resistor_THT:R_Axial_DIN0204_L3.6mm_D1.6mm_P7.62mm_Horizontal, F.Cu at (137.2, 82.5)
Connections:
- U7 pad 8: +BATT -> Net-(U7-CH7)
Routing:
- net +BATT: track 39.4 -> 23.8 mm
- net Net-(U7-CH7): track 0.00 -> 9.84 mm
- net Net-(R18-Pad2): track 0.00 -> 2.54 mm
- net Net-(R19-Pad2): track 0.00 -> 2.54 mm
- net Net-(R17-Pad2): track 0.00 -> 2.54 mm
