File: BIT3.kicad_sch (KiCad schematic)
At the start: 48 parts, among them J1 Conn_02x04_Odd_Even, J2 Conn_01x02_Pin, J3 Conn_01x04_Socket, J4 Conn_02x02_Odd_Even, Q1 2SC1815, SW1 SW_SPDT, SW2 SW_Push, SW3 SW_Push, U2 FODM217A, U3 FODM217A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

Commit message: Tr を置き換え
Parts:
- removed Q1: 2SC1815, Package_TO_SOT_THT:TO-92_Inline, symbol Transistor_BJT:2SC1815
- added Q1: BSP89, Package_TO_SOT_THT:TO-220-3_Vertical, symbol Transistor_FET:BSP89
Connections:
- net FET_D: now also Q1.2 (D)
- net GND: now also Q1.3 (S)
- net at R11.2: now also Q1.1 (G)
Changed lines of the file:
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@@
     )
   )
-  (symbol (lib_id "Transistor_BJT:2SC1815") (at 96.52 76.2 0) (unit 1)
+  (symbol (lib_id "Transistor_FET:BSP89") (at 96.52 76.2 0) (unit 1)
     (in_bom yes) (on_board yes) (dnp no) (fields_autoplaced)
-    (property "Reference" "Q1" (at 101.6 75.565 0)
+    (property "Reference" "Q1" (at 102.87 74.93 0)
       (effects (font (size 1.27 1.27)) (justify left))
     )
-    (property "Value" "2SC1815" (at 101.6 78.105 0)
+    (property "Value" "BSP89" (at 102.87 77.47 0)
       (effects (font (size 1.27 1.27)) (justify left))
     )
-    (property "Footprint" "Package_TO_SOT_THT:TO-92_Inline" (at 101.6 78.105 0)
+    (property "Footprint" "Package_TO_SOT_THT:TO-220-3_Vertical" (at 101.6 78.105 0)
       (effects (font (size 1.27 1.27) italic) (justify left) hide)
     )
-    (property "Datasheet" "https://media.digikey.com/pdf/Data%20Sheets/Toshiba%20PDFs/2SC1815.pdf" (at 96.52 76.2 0)
+    (property "Datasheet" "https://www.infineon.com/dgdl/Infineon-BSP89-DS-v02_02-en.pdf?fileId=db3a30433b47825b013b4b8a07f90d55" (at 96.52 76.2 0)
       (effects (font (size 1.27 1.27)) (justify left) hide)
     )
